File: Hardware/STM32 PIR Sensor.kicad_pcb (KiCad board)
At the start: 2 copper layers, 43.5 x 71 mm, 59 parts, among them J1 Screw_Terminal_01x02, J2 SMA Edge Mount, J3 Conn_01x05_Male, U1 AP62250Z6, U10 LD2410, U2 RFM69HCW, U3 LM75B, U4 STM32L010K8T6, U5 D203S, U6 LM358, U7 LM393

Commit message: v1.2.0. Prototype schematic correction
Parts:
- J2: footprint Connector_Coaxial:SMA_Amphenol_132289_EdgeMount -> Connector_Coaxial:SMA_Samtec_SMA-J-P-X-ST-EM1_EdgeMount
- moved R15 9.66 mm to (249.9, 75.9)
- moved C5 9.24 mm to (239.0, 76.2)
- moved C3 9.24 mm to (241.3, 76.2)
- moved R2 7.92 mm to (248.9, 78.7), turned to 0 degrees
- moved C1 6.70 mm to (241.6, 80.3), turned to -90 degrees
- moved C2 6.10 mm to (248.2, 75.9)
- moved L1 1.02 mm to (244.9, 75.2), turned to 180 degrees
- moved J2 0.67 mm to (230.4, 33.7), turned to 180 degrees
- moved R3 0.25 mm to (245.1, 81.0), turned to 180 degrees
- turned U1 to 0 degrees
Connections:
- U1 pad 1: +12V -> GND
- U1 pad 3: GND -> +12V
- U1 pad 4: Net-(C2-Pad1) -> Net-(R2-Pad1)
- U1 pad 6: Net-(R2-Pad1) -> Net-(C2-Pad1)
Routing:
- net +3.3V: track 128.4 -> 125.4 mm
- net GND: track 1.60 -> 0.10 mm, vias 103 -> 101
- net +12V: track 76.9 -> 78.2 mm
- net Net-(C2-Pad2): track 5.46 -> 6.43 mm
- net Net-(R15-Pad1): track 2.45 -> 1.86 mm
