File: Hardware/STM32 PIR Sensor.kicad_sch (KiCad schematic)
At the start: 28 parts

Commit message: v0.1 Schematic
Parts:
- removed C? (x2): 30p, symbol Device:C
- removed R?: 10k, symbol Device:R
- removed SW?: SW_Push, symbol Switch:SW_Push
- removed Y?: 16 MHz, symbol Device:Crystal
- added C?: 100n, symbol Device:C
- added R? (x2): 10k, symbol Device:R
- added U?: LM75B, symbol Sensor_Temperature:LM75B
Connections:
- net BOOT is gone; now on net +3.3V: U?.31 (BOOT0)
- net +3.3V: now also J?.3 (Pin_3), C?.1, C?.2, R?.1, R?.1, U?.4 (GND), U?.5 (A2), U?.6 (A1), U?.7 (A0), U?.8 (+Vs); no longer J?.5 (Pin_5)
- net NRST: now also J?.5 (Pin_5); no longer J?.4 (Pin_4)
- net SWCLK: now also J?.2 (Pin_2); no longer J?.3 (Pin_3)
- net SWDIO: now also J?.4 (Pin_4); no longer J?.2 (Pin_2)
- net SCL: now reaches U?.29 (PB6)
- net SCL: now also R?.2, U?.2 (SCL)
- net SDA: now reaches U?.30 (PB7)
- net SDA: now also R?.2, U?.1 (SDA)
- no-connect marks 18 -> 19
Other:
- note added: "Temperature Sensor"

Commit message: v0.2 BOM
Parts:
- C1, C10, C11, C12, C2, C3, C4, C5, C6, C7, C8, C9: renamed from C?; footprint (none) -> Capacitor_SMD:C_0805_2012Metric_Pad1.18x1.45mm_HandSolder
- D1: renamed from D?; value D_Schottky -> 1PS70SB10; footprint (none) -> Package_TO_SOT_SMD:SOT-323_SC-70_Handsoldering
- FB1: renamed from FB?; value FerriteBead -> BLM21AG102SN1D; footprint (none) -> Inductor_SMD:L_0805_2012Metric_Pad1.05x1.20mm_HandSolder
- J1: renamed from J?; footprint (none) -> TerminalBlock_Phoenix:TerminalBlock_Phoenix_MKDS-1,5-2_1x02_P5.00mm_Horizontal
- J2: renamed from J?; value Conn_Coaxial -> U.FL-R-SMT-1; footprint (none) -> Connector_Coaxial:U.FL_Hirose_U.FL-R-SMT-1_Vertical
- J3: renamed from J?; footprint (none) -> Connector_PinHeader_2.54mm:PinHeader_1x05_P2.54mm_Horizontal
- L1: renamed from L?; footprint (none) -> Inductor_SMD:L_0805_2012Metric_Pad1.05x1.20mm_HandSolder
- R1, R4: renamed from R?; value 10k -> 4k7; footprint (none) -> Resistor_SMD:R_0805_2012Metric_Pad1.20x1.40mm_HandSolder
- R2, R3: renamed from R?; footprint (none) -> Resistor_SMD:R_0805_2012Metric_Pad1.20x1.40mm_HandSolder
- U1: renamed from U?; footprint Package_TO_SOT_SMD:SOT-563 -> Package_TO_SOT_SMD:TSOT-23-6
- U2: renamed from U?; footprint (none) -> Local:RFM69HCW-XXXS2
- U3: renamed from U?; footprint (none) -> Package_SO:SO-8_5.3x6.2mm_P1.27mm
- U4: renamed from U?; footprint LQFP32_7X7X1P4 -> Package_QFP:LQFP-32_7x7mm_P0.8mm
Connections:
- net PIR0_OUT: now also U4.6 (PA0); no longer U4.18 (PA8)
- net PIR1_OUT: now also U4.8 (PA2); no longer U4.19 (PA9)
- net RF_DIO0: now also U4.19 (PA9); no longer U4.9 (PA3)
- net RF_RESET: now also U4.18 (PA8); no longer U4.8 (PA2)
Other:
- moved on the sheet: C7, D1, FB1, J3, U4A

Commit message: v1.0 with issues
Parts:
- added H1: MountingHole, MountingHole:MountingHole_5mm, symbol Mechanical:MountingHole
- added JP1: Jumper_2_Open, Jumper:SolderJumper-2_P1.3mm_Open_TrianglePad1.0x1.5mm, symbol Jumper:Jumper_2_Open
- added R15: 1k6, Resistor_SMD:R_0603_1608Metric_Pad0.98x0.95mm_HandSolder, symbol Device:R
- added U10: LD2410, Local:LD2410, symbol mmWave_Radar:LD2410
- C1, C10, C11, C12, C2, C4, C6, C7, C8, C9: footprint Capacitor_SMD:C_0805_2012Metric_Pad1.18x1.45mm_HandSolder -> Capacitor_SMD:C_0603_1608Metric_Pad1.08x0.95mm_HandSolder
- D1: value 1PS70SB10 -> STPS0520Z; footprint Package_TO_SOT_SMD:SOT-323_SC-70_Handsoldering -> Diode_SMD:D_SOD-123
- J1: footprint TerminalBlock_Phoenix:TerminalBlock_Phoenix_MKDS-1,5-2_1x02_P5.00mm_Horizontal -> Local:DG301R-5.0
- J2: value U.FL-R-SMT-1 -> SMA Edge Mount; footprint Connector_Coaxial:U.FL_Hirose_U.FL-R-SMT-1_Vertical -> Connector_Coaxial:SMA_Amphenol_132289_EdgeMount
- J3: footprint Connector_PinHeader_2.54mm:PinHeader_1x05_P2.54mm_Horizontal -> Connector_PinHeader_2.54mm:PinHeader_1x05_P2.54mm_Vertical
- R1, R3, R4: footprint Resistor_SMD:R_0805_2012Metric_Pad1.20x1.40mm_HandSolder -> Resistor_SMD:R_0603_1608Metric_Pad0.98x0.95mm_HandSolder
- R2: value 31.6k -> 30k; footprint Resistor_SMD:R_0805_2012Metric_Pad1.20x1.40mm_HandSolder -> Resistor_SMD:R_0603_1608Metric_Pad0.98x0.95mm_HandSolder
Connections:
- net +12V: now also C1.1, D1.1 (K), U1.1 (VIN), JP1.1 (A)
- net +3.3V: now also R15.2; no longer C1.2, C10.2, C11.2, C12.2, C3.2, C4.1, C5.2, C6.2, C7.1, C8.2, C9.2, J1.2 (Pin_2), J2.2 (Ext), J3.3 (Pin_3), R2.1, R3.2, U1.3 (GND), U2.1 (GND), U2.10 (GND), U2.8 (GND), U3.4 (GND), U3.5 (A2), U3.6 (A1), U3.7 (A0), U4.16 (VSS), U4.31 (BOOT0), U4.32 (VSS)
- net PIR0_OUT: now also U4.21 (PA11); no longer U4.6 (PA0)
- net PIR1_OUT: now also U4.22 (PA12); no longer U4.8 (PA2)
- net at R3.1, U1.6 (FB): now also R2.1; no longer R2.2
- net Radar_OUT: now reaches U4.7 (PA1)
- net Radar_OUT: now also U10.5 (OUT)
- net UART_Rx: now reaches U4.9 (PA3)
- net UART_Rx: now also U10.4 (Tx)
- net SP1_MISO renamed SPI_MISO
- net SP1_MOSI renamed SPI_MOSI
- net SP1_NSS renamed SPI_NSS
- net SP1_SCK renamed SPI_SCK
- new net: R15.1, R2.2
- new net: JP1.2 (B), U10.1 (VCC)
- new net GND: C1.2, C10.2, C11.2, C12.2, C3.2, C4.1, C5.2, C6.2, C7.1, C8.2, C9.2, J1.2 (Pin_2), J2.2 (Ext), J3.3 (Pin_3), R3.2, U1.3 (GND), U10.2 (GND), U2.1 (GND), U2.10 (GND), U2.8 (GND), U3.4 (GND), U3.5 (A2), U3.6 (A1), U3.7 (A0), U4.16 (VSS), U4.31 (BOOT0), U4.32 (VSS)
- new net UART_Tx: U10.3 (Rx), U4.8 (PA2)
- no-connect marks 19 -> 17
Other:
- note added: "24GHz mmWave Sensor"
- note added: "Mounting Hole"
- moved on the sheet: J1, L1

Commit message: v1.2.0. Prototype schematic correction
Parts:
- removed C4: 100n, Capacitor_SMD:C_0603_1608Metric_Pad1.08x0.95mm_HandSolder, symbol Device:C
- removed J3: Conn_01x05_Male, Connector_PinHeader_2.54mm:PinHeader_1x05_P2.54mm_Vertical, symbol Connector:Conn_01x05_Male
- removed R1, R4: 4k7, Resistor_SMD:R_0603_1608Metric_Pad0.98x0.95mm_HandSolder, symbol Device:R
- removed U3: LM75B, Package_SO:SO-8_5.3x6.2mm_P1.27mm, symbol Sensor_Temperature:LM75B
- added C23: 100n, Capacitor_SMD:C_0603_1608Metric_Pad1.08x0.95mm_HandSolder, symbol Device:C
- added D3: LL-S170PVC-V1-2B, LED_SMD:LED_0805_2012Metric_Pad1.15x1.40mm_HandSolder, symbol Device:LED
- added J4: Conn_02x05_Odd_Even, Connector_IDC:IDC-Header_2x05_P2.54mm_Vertical, symbol Connector_Generic:Conn_02x05_Odd_Even
- added JP2: SolderJumper_2_Open, symbol Jumper:SolderJumper_2_Open
- added R16: 62, Resistor_SMD:R_0603_1608Metric_Pad0.98x0.95mm_HandSolder, symbol Device:R
- H1: value MountingHole -> PIR Lens Mounting; footprint MountingHole:MountingHole_5mm -> Local:PIR_Mounting
Connections:
- net +12V: now also U1.3 (VIN); no longer U1.1 (VIN)
- net +3.3V: now also C23.1, JP2.1 (A)
- net GND: now also U1.1 (GND), C23.2, D3.1 (K), J4.3 (Pin_3), J4.4 (Pin_4); no longer U1.3 (GND)
- net NRST: now also J4.1 (Pin_1)
- net SWCLK: now also J4.6 (Pin_6)
- net SWDIO: now also J4.2 (Pin_2)
- net at R2.1, R3.1: now also U1.4 (FB); no longer U1.6 (FB)
- net at C2.1: now also U1.6 (BST); no longer U1.4 (BST)
- net LED: now reaches U4.20 (PA10)
- net LED: now also R16.1
- net SCL: no longer names the net of U4.29 (PB6)
- net SDA: no longer names the net of U4.30 (PB7)
- new net: D3.2 (A), R16.2
- new net: J4.7 (Pin_7), J4.8 (Pin_8), JP2.2 (B)
- no-connect marks 17 -> 20
Other:
- note removed: "Temperature Sensor"
- moved on the sheet: H1
