File: Hardware/pir_sensor.kicad_sch (KiCad schematic)
At the start: 34 parts

Commit message: v0.2 BOM
Parts:
- C13, C15, C16, C17, C18, C19, C20, C21, C22: renamed from C?; footprint (none) -> Capacitor_SMD:C_0805_2012Metric_Pad1.18x1.45mm_HandSolder
- C14: renamed from C?; footprint (none) -> Capacitor_SMD:CP_Elec_6.3x5.4
- D2: renamed from D?; footprint Diode_THT:D_DO-35_SOD27_P7.62mm_Horizontal -> Diode_SMD:D_0805_2012Metric_Pad1.15x1.40mm_HandSolder
- R10, R11, R12, R13, R14, R15, R16, R17, R18, R5, R6, R7, R8, R9: renamed from R?; footprint (none) -> Resistor_SMD:R_0805_2012Metric_Pad1.20x1.40mm_HandSolder
- U5: renamed from U?; footprint (none) -> Package_TO_SOT_THT:TO-5-3
- U6, U7: renamed from U?; footprint (none) -> Package_SO:SO-8_5.3x6.2mm_P1.27mm
- gave numbers to parts that had none: 2

Commit message: v1.0 with issues
Parts:
- removed R15, R16: 470, Resistor_SMD:R_0805_2012Metric_Pad1.20x1.40mm_HandSolder, symbol Device:R
- removed U8, U9: LTV-357T, Package_SO:SO-4_4.4x3.6mm_P2.54mm, symbol Isolator:LTV-357T
- added TP1: Analog PIR, TestPoint:TestPoint_Pad_D1.0mm, symbol Connector:TestPoint
- added TP2: Digital PIR_H, TestPoint:TestPoint_Pad_D1.0mm, symbol Connector:TestPoint
- added TP3: Digital PIR_L, TestPoint:TestPoint_Pad_D1.0mm, symbol Connector:TestPoint
- C13, C16, C18, C19, C20, C21, C22: footprint Capacitor_SMD:C_0805_2012Metric_Pad1.18x1.45mm_HandSolder -> Capacitor_SMD:C_0603_1608Metric_Pad1.08x0.95mm_HandSolder
- D2: footprint Diode_SMD:D_0805_2012Metric_Pad1.15x1.40mm_HandSolder -> Diode_SMD:D_MiniMELF
- R10, R11, R12, R13, R14, R5, R6, R7, R8, R9: footprint Resistor_SMD:R_0805_2012Metric_Pad1.20x1.40mm_HandSolder -> Resistor_SMD:R_0603_1608Metric_Pad0.98x0.95mm_HandSolder
- R17, R18: value 1k -> 4k7; footprint Resistor_SMD:R_0805_2012Metric_Pad1.20x1.40mm_HandSolder -> Resistor_SMD:R_0603_1608Metric_Pad0.98x0.95mm_HandSolder
Connections:
- net PIR_OUT_H: now also U7.1, TP2.1
- net PIR_OUT_L: now also U7.7, TP3.1
- net at C19.2, R10.2, U6.7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: now also TP1.1
Other:
- moved on the sheet: R17, R18

Commit message: v0.0.3(1) PIR&RFM69
Parts:
- added RV?: 5k, symbol Device:R_Potentiometer
- R9: value 12k -> 7k
Connections:
- net GND: now also RV?.3
- net at C19.1, R10.1, U6.6 (-): now also RV?.2; no longer R9.2
- new net: R9.2, RV?.1
Other:
- moved on the sheet: C18, C19, C21, R10, R11, R12, R13, R14, R17, R18, R9, TP1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

Commit message: v1.2.0. Prototype schematic correction
Parts:
- removed RV?: 5k, symbol Device:R_Potentiometer
- added PS-6: 1M, Local:Potentiometer_PS-6_Vertical_Hole, symbol Device:R_Potentiometer
Connections:
- net GND: now also PS-6.3
- net at C19.1, R10.1, U6.6 (-): now also R9.2
- net at C19.2, TP1.1, U6.7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: now also PS-6.2; no longer R10.2
- new net: PS-6.1, R10.2
Other:
- moved on the sheet: C19, R10
